Commit message: modify xacro to get front wheel rotation

File: ros2_ws/src/car_like_mobile_robot_description/urdf/include/gazebo_plugin.xacro (robot description, xacro)
@@ -8,4 +8,11 @@
     </plugin>
   </gazebo>
+  <plugin filename="libgazebo_ros_pose.so" name="gazebo_ros_pose">
+    <ros>
+      <namespace>/car_like_mobile_robot</namespace>
+      <remapping>pose:=odom</remapping>
+    </ros>
+    <update_rate>50</update_rate>
+  </plugin>
   <!-- IMU PLUGIN  -->
   <!-- <gazebo reference="imu_link">

File: ros2_ws/src/car_like_mobile_robot_description/urdf/include/ros2_control.xacro (robot description, xacro)
@@ -6,5 +6,5 @@
       </hardware>
       <!-- 前輪の車輪（受動車輪） -->
-      <!-- <joint name="vehicle_front_left_joint">
+      <joint name="vehicle_front_left_joint">
         <command_interface name="effort">
           <param name="min">0.0</param>
@@ -16,12 +16,12 @@
       </joint>
       <joint name="vehicle_front_right_joint">
-        <command_interface name="velocity">
-          <param name="min">-6.28</param>
-          <param name="max">6.28</param>
+        <command_interface name="effort">
+          <param name="min">0.0</param>
+          <param name="max">0.0</param>
         </command_interface>
         <state_interface name="position"/>
         <state_interface name="velocity"/>
         <state_interface name="effort"/>
-      </joint> -->
+      </joint>
       <!-- 前輪ステアリング -->
       <joint name="vehicle_front_left_steering_joint">
